File: 02_Assemble/GS84.kicad_pcb (KiCad board)
At the start: 2 copper layers, 304.4 x 98.8 mm, 150 parts, among them J1 Conn_01x02, SW1 SW_PUSH, SW10 SW_PUSH, SW11 SW_PUSH, SW12 SW_PUSH, SW13 SW_PUSH, SW14 SW_PUSH, SW15 SW_PUSH, SW16 SW_PUSH, SW17 SW_PUSH, SW18 SW_PUSH, SW19 SW_PUSH, SW2 SW_PUSH, SW20 SW_PUSH, SW21 SW_PUSH, SW22 SW_PUSH, SW23 SW_PUSH, SW24 SW_PUSH, SW25 SW_PUSH, SW26 SW_PUSH, SW27 SW_PUSH, SW28 SW_PUSH, SW29 SW_PUSH, SW3 SW_PUSH, SW30 SW_PUSH, SW31 SW_PUSH, SW32 SW_PUSH, SW33 SW_PUSH, SW34 SW_PUSH, SW35 SW_PUSH, SW36 SW_PUSH, SW37 SW_PUSH, SW38 SW_PUSH, SW39 SW_PUSH, SW4 SW_PUSH, SW40 SW_PUSH, SW41 SW_PUSH, SW42 SW_PUSH, SW43 SW_PUSH, SW44 SW_PUSH, SW45 SW_PUSH, SW46 SW_PUSH, SW47 SW_PUSH, SW48 SW_PUSH, SW49 SW_PUSH, SW5 SW_PUSH, SW50 SW_PUSH, SW6 SW_PUSH, SW7 SW_PUSH, SW8 SW_PUSH, SW9 SW_PUSH, U1 BLEMicroPro

Commit message: レビューいただいた内容を反映
ProMicoroを中央に移動、ダイオードを表面実装だけに修正、バッテリーホールと信号線の距離を広げる
Parts:
- D1, D10, D11, D12, D13, D14, D15, D16, D17, D18, D19, D2, D20, D21, D22, D23, D24, D25, D26, D27, D28, D29, D3, D30, D31, D32, D33, D34, D35, D36, D37, D38, D39, D4, D40, D41, D42, D43, D44, D45, D46, D47, D48, D49, D5, D6, D7, D8, D9: footprint kbd_Parts:Diode_TH_SMD -> kbd_Parts:Diode_SMD
- SW24: footprint kbd_SW:CherryMX_Hotswap_1u -> kbd_SW:CherryMX_Hotswap_1u_Small1
- SW37: footprint kbd_SW:CherryMX_Hotswap_1u_Small1 -> kbd_SW:CherryMX_Hotswap_1u
- moved SW50 141.4 mm to (151.2, 41.7), turned to 0 degrees
- moved U1 106.6 mm to (164.3, 30.4)
- moved L49 68.2 mm to (300.0, 38.1)
- moved L32 67.6 mm to (212.5, 38.1)
- moved L29 67.1 mm to (200.6, 104.8)
- moved L45 67.1 mm to (292.3, 104.8)
- moved L40 67.0 mm to (250.6, 38.1), turned to 5 degrees
- moved L37 66.8 mm to (254.2, 104.8), turned to 0 degrees
- moved L12 66.7 mm to (92.9, 104.8), turned to 0 degrees
- moved L5 66.7 mm to (54.8, 104.8), turned to 0 degrees
- moved L15 66.7 mm to (92.3, 38.1), turned to 355 degrees
- moved L8 66.1 mm to (54.8, 38.1), turned to 355 degrees
- moved L20 62.6 mm to (142.9, 99.4), turned to 265 degrees
- moved L23 62.6 mm to (130.4, 38.1), turned to 355 degrees
- moved L48 45.8 mm to (302.4, 59.5)
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Routing:
- net VCC: track 1381.4 -> 1849.9 mm, vias 34 -> 0
- net GND: track 1404.7 -> 1703.7 mm, vias 48 -> 49
- net Col0: track 477.1 -> 352.3 mm, vias 11 -> 9
- net Net-(L44-Pad1): track 98.7 -> 15.4 mm, vias 2 -> 0
- net Col2: track 396.8 -> 314.0 mm, vias 11 -> 9
- net Net-(L19-Pad1): track 99.6 -> 20.3 mm, vias 4 -> 2
- net Net-(L32-Pad1): track 92.8 -> 15.8 mm, vias 2 -> 0
- net Col3: track 418.1 -> 344.4 mm, vias 14 -> 10
- net Col4: track 429.5 -> 355.9 mm, vias 13 -> 10
- net Col1: track 423.0 -> 351.0 mm, vias 14 -> 10
- net Net-(L40-Pad1): track 86.5 -> 14.8 mm, vias 4 -> 0
- net LED: track 233.2 -> 163.6 mm, vias 1 -> 3
- net Net-(L28-Pad1): track 93.6 -> 25.3 mm, vias 4 -> 0
- net Net-(L8-Pad1): track 81.5 -> 14.5 mm, vias 2 -> 0
- net Net-(L15-Pad1): track 77.4 -> 14.6 mm, vias 4 -> 0
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